File: shield_gas_sensor/shield_gas_sensor.kicad_pcb (KiCad board)
At the start: 2 copper layers, 68.6 x 53.3 mm, 8 parts, among them P1 Power, P2 Analog, P3 Digital, P4 Digital, P5 CONN_01X01, P6 CONN_01X01, P7 CONN_01X01, P8 CONN_01X01

Commit message: Placement composants
Parts:
- added C1: 100n, Capacitor_THT:CP_Radial_D4.0mm_P1.50mm, F.Cu at (126.2, 113.7)
- added C2: 100n, Capacitor_THT:CP_Radial_D4.0mm_P1.50mm, F.Cu at (166.9, 101.0)
- added C3: 100n, Capacitor_THT:CP_Radial_D4.0mm_P1.50mm, F.Cu at (156.7, 117.5)
- added C4: 1u, Capacitor_THT:CP_Radial_D4.0mm_P1.50mm, F.Cu at (159.3, 97.2)
- added R1: 100k, Resistor_THT:R_Axial_DIN0204_L3.6mm_D1.6mm_P5.08mm_Horizontal, F.Cu at (133.9, 84.5)
- added R3: 100k, Resistor_THT:R_Axial_DIN0204_L3.6mm_D1.6mm_P5.08mm_Horizontal, F.Cu at (151.6, 104.8)
- added R5: 10k, Resistor_THT:R_Axial_DIN0204_L3.6mm_D1.6mm_P5.08mm_Horizontal, F.Cu at (144.0, 84.5)
- added R6: 1k, Resistor_THT:R_Axial_DIN0204_L3.6mm_D1.6mm_P5.08mm_Horizontal, F.Cu at (166.9, 85.7)
- added Rcal1: R, Resistor_THT:R_Axial_DIN0204_L3.6mm_D1.6mm_P5.08mm_Horizontal, F.Cu at (121.2, 101.0)
- added Rcal2: R, Resistor_THT:R_Axial_DIN0204_L3.6mm_D1.6mm_P5.08mm_Horizontal, F.Cu at (116.1, 106.0)
- added Rsensor1: R, EmpreintesCapGaz:TO-5-4_cap_gaz, F.Cu at (147.8, 95.9)
- added U1: LTC1050, Package_DIP:DIP-8_W7.62mm_LongPads, F.Cu at (130.0, 98.4)
