File: shield_gas_sensor/shield_gas_sensor.kicad_pcb (KiCad board)
At the start: 2 copper layers, 68.6 x 53.3 mm, 20 parts, among them P1 Power, P2 Analog, P3 Digital, P4 Digital, P5 CONN_01X01, P6 CONN_01X01, P7 CONN_01X01, P8 CONN_01X01, U1 LTC1050

Commit message: Placement composants 2
Connections:
- P2 pad 5: /A4(SDA) -> Net-(P2-Pad5)
- P2 pad 6: /A5(SCL) -> Net-(P2-Pad6)
Changed lines of the file:
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@@
     (zones 0)
     (modules 20)
-    (nets 41)
+    (nets 43)
   )
   (page A4)
@@
   (net 39 "Net-(U1-Pad5)")
   (net 40 "Net-(U1-Pad8)")
+  (net 41 "Net-(P2-Pad5)")
+  (net 42 "Net-(P2-Pad6)")
   (net_class Default "This is the default net class."
     (clearance 0.2)
@@
     (add_net "Net-(C4-Pad2)")
     (add_net "Net-(P1-Pad1)")
+    (add_net "Net-(P2-Pad5)")
+    (add_net "Net-(P2-Pad6)")
     (add_net "Net-(P5-Pad1)")
     (add_net "Net-(P6-Pad1)")
@@
       (net 9 /A3))
     (pad 5 thru_hole oval (at 10.16 0) (size 1.7272 2.032) (drill 1.016) (layers *.Cu *.Mask F.SilkS)
-      (net 11 "/A4(SDA)"))
+      (net 41 "Net-(P2-Pad5)"))
     (pad 6 thru_hole oval (at 12.7 0) (size 1.7272 2.032) (drill 1.016) (layers *.Cu *.Mask F.SilkS)
-      (net 12 "/A5(SCL)"))
+      (net 42 "Net-(P2-Pad6)"))
     (model ${KIPRJMOD}/Socket_Arduino_Uno.3dshapes/Socket_header_Arduino_1x06.wrl
       (offset (xyz 6.349999904632568 0 0))

Commit message: Fin du PCB
Parts:
- added U2: RN2483_Breakout, MesEmpreinte:RN2483, F.Cu at (188.5, 92.1)
Connections:
- P4 pad 7: /1(Tx) -> /Tx
- P4 pad 8: /0(Rx) -> /Rx
Routing:
- net GND: track 0.00 -> 180.5 mm
- net +3V3: track 0.00 -> 151.0 mm
- net /Reset: track 0.00 -> 103.7 mm
- net Net-(C4-Pad2): track 0.00 -> 72.6 mm
- net /Rx: track 0.00 -> 59.8 mm
- net /A0: track 0.00 -> 40.3 mm
- net Net-(C1-Pad1): track 0.00 -> 39.4 mm
- net Net-(C4-Pad1): track 0.00 -> 39.4 mm
- net +5V: track 0.00 -> 37.0 mm
- net /Tx: track 0.00 -> 32.3 mm
- net Net-(R5-Pad1): track 0.00 -> 14.5 mm
- net Net-(Rcal1-Pad2): track 0.00 -> 5.08 mm
- added copper zone on B.Cu, net (none)
Other:
- board size 68.6 x 53.3 mm -> 132.1 x 63.5 mm
- net class Default: clearance 0.2 -> 0.4; trace_width 0.25 -> 0.8; via_dia 0.6 -> 1.6; via_drill 0.4 -> 0.8
- rule trace_clearance: 0.2 -> 0.4
- rule trace_min: 0.2 -> 0.8
- rule via_min_drill: 0.3 -> 0.8
- rule via_min_size: 0.4 -> 1.6
- board text added: "ALOÏSI-CHASSERAT SHIELD - TOP"
